Commit message: two robots simulation

File: nono_description/urdf/nono.urdf.xacro (robot description, xacro)
@@ -84,5 +84,5 @@
   <!-- Infrared Marker -->
   <xacro:if value="${use_smocap_ir_marker}">
-    <xacro:cs_smocap_ir_marker>
+    <xacro:cs_smocap_ir_marker mesh="${smocap_ir_marker_mesh}">
       <origin xyz="-0.0255 0 0.039" rpy="0 0 0" />
     </xacro:cs_smocap_ir_marker>

File: nono_description/urdf/nono_1.urdf.xacro (robot description, xacro)
@@ -1,8 +1,8 @@
 <?xml version="1.0" encoding="utf8"?>
-<robot name="nono_0" xmlns:xacro="http://www.ros.org/wiki/xacro">
-  <xacro:property name="robot_name" value="nono_0" />
+<robot name="nono_1" xmlns:xacro="http://www.ros.org/wiki/xacro">
+  <xacro:property name="robot_name" value="nono_1" />
   <xacro:property name="use_eachine_camera" value="False" />
   <xacro:property name="use_smocap_ir_marker" value="True" />
-  <xacro:property name="smocap_ir_marker_mesh" value="ir_marker_0.dae" />
+  <xacro:property name="smocap_ir_marker_mesh" value="ir_marker.dae" />
   <!-- dimensions -->
   <xacro:property name="chassis_radius" value="0.04" />
